Commit message: Update URDF

File: qronk_description/urdf/base_qronk.xacro (robot description, xacro)
@@ -1,9 +1,17 @@
 <?xml version="1.0"?>
 <robot xmlns:xacro="http://www.ros.org/wiki/xacro">
-    <link name="base_link">
+    <link name="base_link" />
+    <joint name="base_chassis_joint" type="fixed">
+        <parent link="base_link" />
+        <child link="chassis" />
+        <origin xyz="0 0 0" rpy="${pi / 2.0} 0 0" />
+    </joint>
+    <link name="chassis">
         <visual>
             <geometry>
-                <box size="0.1 0.1 0.1" />
+                <mesh filename="package://qronk_description/meshes/chassis.stl"
+                    scale="0.001 0.001 0.001" />
             </geometry>
+            <origin xyz="-0.047147 0 -0.1075" rpy="0 0 0" />
         </visual>
     </link>

File: qronk_description/urdf/qronk.urdf.xacro (robot description, xacro)
@@ -3,3 +3,4 @@
     <xacro:include filename="common_properties.xacro" />
     <xacro:include filename="base_qronk.xacro" />
+    <!-- <xacro:include filename="leg.xacro" /> -->
 </robot>

Commit message: commit on "main"

File: qronk_description/urdf/base_qronk.xacro (robot description, xacro)
@@ -5,5 +5,5 @@
         <parent link="base_link" />
         <child link="chassis" />
-        <origin xyz="0 0 0" rpy="${pi / 2.0} 0 0" />
+        <origin xyz="0 0 0" rpy="0 0 0" />
     </joint>
     <link name="chassis">
@@ -13,5 +13,6 @@
                     scale="0.001 0.001 0.001" />
             </geometry>
-            <origin xyz="-0.047147 0 -0.1075" rpy="0 0 0" />
+            <origin xyz="0 0 0" rpy="0 0 0" />
+            <material name="grey" />
         </visual>
     </link>

File: qronk_description/urdf/common_properties.xacro (robot description, xacro)
@@ -1,3 +1,15 @@
 <?xml version="1.0"?>
 <robot xmlns:xacro="http://www.ros.org/wiki/xacro">
+    <material name="red">
+        <color rgba="0.5 0 0 1" />
+    </material>
+    <material name="green">
+        <color rgba="0 0.5 0 1" />
+    </material>
+    <material name="blue">
+        <color rgba="0 0 0.5 1" />
+    </material>
+    <material name="grey">
+        <color rgba="0.5 0.5 0.5 1" />
+    </material>
 </robot>

Commit message: Update URDF

File: qronk_description/urdf/base_qronk.xacro (robot description, xacro)
@@ -1,9 +1,8 @@
 <?xml version="1.0"?>
 <robot xmlns:xacro="http://www.ros.org/wiki/xacro">
-    <link name="base_link" />
     <joint name="base_chassis_joint" type="fixed">
         <parent link="base_link" />
         <child link="chassis" />
-        <origin xyz="0 0 0" rpy="0 0 0" />
+        <origin xyz="0 0 0.038144" rpy="0 0 0" />
     </joint>
     <link name="chassis">
@@ -16,4 +15,66 @@
             <material name="grey" />
         </visual>
+        <!-- TODO will have collision with its own components; needs fix -->
+        <collision>
+            <geometry>
+                <box size="0.185 0.136835 0.000495" />
+            </geometry>
+            <origin xyz="0 0 0" rpy="0 0 0" />
+        </collision>
+        <!-- numbers are based on Fusion 360 calculations -->
+        <inertial>
+            <mass value="0.345" />
+            <inertia ixx="1.452E-3" ixy="-1.094E-3" ixz="-1.442E-4"
+                iyy="2.678E-3" iyz="-1.244E-4"
+                izz="3.674E-3" />
+        </inertial>
+    </link>
+    <joint name="chassis_battery_joint" type="fixed">
+        <parent link="chassis" />
+        <child link="battery" />
+        <origin xyz="0 0 -0.0305" rpy="0 0 0" />
+    </joint>
+    <link name="battery">
+        <visual>
+            <geometry>
+                <mesh filename="package://qronk_description/meshes/battery.stl"
+                    scale="0.001 0.001 0.001" />
+            </geometry>
+            <origin xyz="-0.069 -0.0225 0" rpy="0 0 0" />
+            <material name="grey" />
+        </visual>
+        <collision>
+            <geometry>
+                <box size="0.138 0.045 0.018" />
+            </geometry>
+            <origin xyz="-0.069 -0.0225 0" rpy="0 0 0" />
+        </collision>
+        <!-- TODO simple approximation; needs correction -->
+        <xacro:box_inertia m="0.15" l="0.138" w="0.045" h="0.018"
+            xyz="-0.069 -0.0225 0" rpy="0 0 0" />
+    </link>
+    <joint name="chassis_raspberry_joint" type="fixed">
+        <parent link="chassis" />
+        <child link="raspberry_link" />
+        <origin xyz="0 0 0.044" rpy="0 0 0" />
+    </joint>
+    <link name="raspberry_link">
+        <visual>
+            <geometry>
+                <mesh filename="package://qronk_description/meshes/raspberry.stl"
+                    scale="0.001 0.001 0.001" />
+            </geometry>
+            <origin xyz="-0.05 -0.035 0" rpy="0 0 0" />
+            <material name="grey" />
+        </visual>
+        <collision>
+            <geometry>
+                <box size="0.1 0.07 0.025" />
+            </geometry>
+            <origin xyz="-0.05 -0.035 0" rpy="0 0 0" />
+        </collision>
+        <!-- TODO simple approximation, needs correction -->
+        <xacro:box_inertia m="0.35" l="0.1" w="0.07" h="0.025"
+            xyz="-0.05 -0.035 0" rpy="0 0 0" />
     </link>
 </robot>

File: qronk_description/urdf/qronk.urdf.xacro (robot description, xacro)
@@ -1,4 +1,5 @@
 <?xml version="1.0"?>
 <robot name="qronk" xmlns:xacro="http://www.ros.org/wiki/xacro">
+    <link name="base_link" />
     <xacro:include filename="common_properties.xacro" />
     <xacro:include filename="base_qronk.xacro" />
