Commit message: Add foot to URDF

File: qronk_description/urdf/leg_BL.xacro (robot description, xacro)
@@ -52,3 +52,17 @@
         </visual>
     </link>
+    <joint name="lower_leg_foot_BL_joint" type="fixed">
+        <parent link="lower_leg_BL_link" />
+        <child link="foot_BL_link" />
+        <origin xyz="-0 0.0066835 -0.09416" rpy="0 0 0" />
+    </joint>
+    <link name="foot_BL_link">
+        <visual>
+            <geometry>
+                <sphere radius="0.0075" />
+            </geometry>
+            <origin xyz="0 0 0" rpy="0 0 0" />
+            <material name="grey" />
+        </visual>
+    </link>
 </robot>

File: qronk_description/urdf/leg_BL_gazebo.xacro (robot description, xacro)
@@ -10,3 +10,6 @@
         <material>Gazebo/Grey</material>
     </gazebo>
+    <gazebo reference="foot_BL_link">
+        <material>Gazebo/Grey</material>
+    </gazebo>
 </robot>

File: qronk_description/urdf/leg_BR.xacro (robot description, xacro)
@@ -52,3 +52,17 @@
         </visual>
     </link>
+    <joint name="lower_leg_foot_BR_joint" type="fixed">
+        <parent link="lower_leg_BR_link" />
+        <child link="foot_BR_link" />
+        <origin xyz="-0 -0.0066835 -0.09416" rpy="0 0 0" />
+    </joint>
+    <link name="foot_BR_link">
+        <visual>
+            <geometry>
+                <sphere radius="0.0075" />
+            </geometry>
+            <origin xyz="0 0 0" rpy="0 0 0" />
+            <material name="grey" />
+        </visual>
+    </link>
 </robot>

File: qronk_description/urdf/leg_BR_gazebo.xacro (robot description, xacro)
@@ -10,3 +10,6 @@
         <material>Gazebo/Grey</material>
     </gazebo>
+    <gazebo reference="foot_BR_link">
+        <material>Gazebo/Grey</material>
+    </gazebo>
 </robot>

File: qronk_description/urdf/leg_FL.xacro (robot description, xacro)
@@ -52,3 +52,17 @@
         </visual>
     </link>
+    <joint name="lower_leg_foot_FL_joint" type="fixed">
+        <parent link="lower_leg_FL_link" />
+        <child link="foot_FL_link" />
+        <origin xyz="0 0.0066835 -0.09416" rpy="0 0 0" />
+    </joint>
+    <link name="foot_FL_link">
+        <visual>
+            <geometry>
+                <sphere radius="0.0075" />
+            </geometry>
+            <origin xyz="0 0 0" rpy="0 0 0" />
+            <material name="grey" />
+        </visual>
+    </link>
 </robot>

File: qronk_description/urdf/leg_FL_gazebo.xacro (robot description, xacro)
@@ -10,3 +10,6 @@
         <material>Gazebo/Grey</material>
     </gazebo>
+    <gazebo reference="foot_FL_link">
+        <material>Gazebo/Grey</material>
+    </gazebo>
 </robot>

File: qronk_description/urdf/leg_FR.xacro (robot description, xacro)
@@ -52,3 +52,17 @@
         </visual>
     </link>
+    <joint name="lower_leg_foot_FR_joint" type="fixed">
+        <parent link="lower_leg_FR_link" />
+        <child link="foot_FR_link" />
+        <origin xyz="0 -0.0066835 -0.09416" rpy="0 0 0" />
+    </joint>
+    <link name="foot_FR_link">
+        <visual>
+            <geometry>
+                <sphere radius="0.0075" />
+            </geometry>
+            <origin xyz="0 0 0" rpy="0 0 0" />
+            <material name="grey" />
+        </visual>
+    </link>
 </robot>

File: qronk_description/urdf/leg_FR_gazebo.xacro (robot description, xacro)
@@ -10,3 +10,6 @@
         <material>Gazebo/Grey</material>
     </gazebo>
+    <gazebo reference="foot_FR_link">
+        <material>Gazebo/Grey</material>
+    </gazebo>
 </robot>
