Commit message: Update URDF

File: qronk_description/urdf/chassis.xacro (robot description, xacro)
@@ -3,8 +3,8 @@
     <joint name="base_chassis_joint" type="fixed">
         <parent link="base_link" />
-        <child link="chassis" />
+        <child link="chassis_link" />
         <origin xyz="0 0 0.038144" rpy="0 0 0" />
     </joint>
-    <link name="chassis">
+    <link name="chassis_link">
         <visual>
             <geometry>
@@ -31,9 +31,9 @@
     </link>
     <joint name="chassis_battery_joint" type="fixed">
-        <parent link="chassis" />
-        <child link="battery" />
+        <parent link="chassis_link" />
+        <child link="battery_link" />
         <origin xyz="0 0 -0.0305" rpy="0 0 0" />
     </joint>
-    <link name="battery">
+    <link name="battery_link">
         <visual>
             <geometry>
@@ -55,5 +55,5 @@
     </link>
     <joint name="chassis_raspberry_joint" type="fixed">
-        <parent link="chassis" />
+        <parent link="chassis_link" />
         <child link="raspberry_link" />
         <origin xyz="0 0 0.044" rpy="0 0 0" />

File: qronk_description/urdf/qronk.urdf.xacro (robot description, xacro)
@@ -4,4 +4,5 @@
     <xacro:include filename="common_properties.xacro" />
     <xacro:include filename="chassis.xacro" />
+    <xacro:include filename="chassis_gazebo.xacro" />
     <!-- <xacro:include filename="leg.xacro" /> -->
 </robot>

Commit message: Update URDF

File: qronk_description/urdf/chassis.xacro (robot description, xacro)
@@ -18,5 +18,5 @@
         <collision>
             <geometry>
-                <box size="0.185 0.136835 0.000495" />
+                <box size="0.185 0.136835 0.0495" />
             </geometry>
             <origin xyz="0 0 0" rpy="0 0 0" />

Commit message: Update URDF

File: qronk_description/urdf/chassis.xacro (robot description, xacro)
@@ -48,5 +48,5 @@
                 <box size="0.138 0.045 0.018" />
             </geometry>
-            <origin xyz="-0.069 -0.0225 0" rpy="0 0 0" />
+            <origin xyz="0 0 0.009" rpy="0 0 0" />
         </collision>
         <!-- TODO simple approximation; needs correction -->
@@ -72,5 +72,5 @@
                 <box size="0.1 0.07 0.025" />
             </geometry>
-            <origin xyz="-0.05 -0.035 0" rpy="0 0 0" />
+            <origin xyz="0 0 0.0125" rpy="0 0 0" />
         </collision>
         <!-- TODO simple approximation, needs correction -->

Commit message: Update URDF

File: qronk_description/urdf/chassis.xacro (robot description, xacro)
@@ -18,7 +18,7 @@
         <collision>
             <geometry>
-                <box size="0.185 0.136835 0.0495" />
+                <box size="0.185 0.136835 0.084144" />
             </geometry>
-            <origin xyz="0 0 0" rpy="0 0 0" />
+            <origin xyz="0 0 0.003928" rpy="0 0 0" />
         </collision>
         <!-- numbers are based on Fusion 360 calculations -->
@@ -74,5 +74,5 @@
             <origin xyz="0 0 0.0125" rpy="0 0 0" />
         </collision>
-        <!-- TODO simple approximation, needs correction -->
+        <!-- TODO simple approximation; needs correction -->
         <xacro:box_inertia m="0.35" l="0.1" w="0.07" h="0.025"
             xyz="-0.05 -0.035 0" rpy="0 0 0" />

Commit message: Update URDF

File: qronk_description/urdf/chassis.xacro (robot description, xacro)
@@ -4,5 +4,5 @@
         <parent link="base_link" />
         <child link="chassis_link" />
-        <origin xyz="0 0 0.038144" rpy="0 0 0" />
+        <origin xyz="0 0 0" rpy="0 0 0" />
     </joint>
     <link name="chassis_link">

File: qronk_description/urdf/leg.xacro (robot description, xacro)
@@ -1,3 +1,48 @@
 <?xml version="1.0"?>
 <robot xmlns:xacro="http://www.ros.org/wiki/xacro">
+    <joint name="base_shoulder_joint" type="fixed">
+        <parent link="base_link" />
+        <child link="shoulder_link" />
+        <origin xyz="0.0885 -0.047417 0.000052" rpy="0 0 0" />
+    </joint>
+    <link name="shoulder_link">
+        <visual>
+            <geometry>
+                <mesh filename="package://qronk_description/meshes/shoulder.stl"
+                    scale="0.001 0.001 0.001" />
+            </geometry>
+            <origin xyz="0 0 0" rpy="0 0 0" />
+            <material name="grey" />
+        </visual>
+    </link>
+    <joint name="shoulder_upper_leg_joint" type="fixed">
+        <parent link="shoulder_link" />
+        <child link="upper_leg_link" />
+        <origin xyz="0.03 -0.0214 -0.00002" rpy="0 0 0" />
+    </joint>
+    <link name="upper_leg_link">
+        <visual>
+            <geometry>
+                <mesh filename="package://qronk_description/meshes/upper_leg.stl"
+                    scale="0.001 0.001 0.001" />
+            </geometry>
+            <origin xyz="0 0 0" rpy="0 0 0" />
+            <material name="grey" />
+        </visual>
+    </link>
+    <joint name="upper_leg_lower_leg_joint" type="fixed">
+        <parent link="upper_leg_link" />
+        <child link="lower_leg_link" />
+        <origin xyz="0 -0.016349 -0.098459" rpy="0 0 0" />
+    </joint>
+    <link name="lower_leg_link">
+        <visual>
+            <geometry>
+                <mesh filename="package://qronk_description/meshes/lower_leg.stl"
+                    scale="0.001 0.001 0.001" />
+            </geometry>
+            <origin xyz="0 0 0" rpy="0 0 0" />
+            <material name="grey" />
+        </visual>
+    </link>
 </robot>

File: qronk_description/urdf/qronk.urdf.xacro (robot description, xacro)
@@ -5,4 +5,5 @@
     <xacro:include filename="chassis.xacro" />
     <xacro:include filename="chassis_gazebo.xacro" />
-    <!-- <xacro:include filename="leg.xacro" /> -->
+    <xacro:include filename="leg.xacro" />
+    <xacro:include filename="leg_gazebo.xacro" />
 </robot>

Commit message: Add collision and inertial values to URDF

File: qronk_description/urdf/chassis.xacro (robot description, xacro)
@@ -15,5 +15,4 @@
             <material name="grey" />
         </visual>
-        <!-- TODO will have collision with its own components; needs fix -->
         <collision>
             <geometry>
@@ -22,11 +21,6 @@
             <origin xyz="0 0 0.003928" rpy="0 0 0" />
         </collision>
-        <!-- numbers are based on Fusion 360 calculations -->
-        <inertial>
-            <mass value="0.345" />
-            <inertia ixx="1.452E-3" ixy="-1.094E-3" ixz="-1.442E-4"
-                iyy="2.678E-3" iyz="-1.244E-4"
-                izz="3.674E-3" />
-        </inertial>
+        <xacro:box_inertia m="0.3" l="0.185" w="0.137" h="0.084"
+            xyz="0 0 0.004" rpy="0 0 0" />
     </link>
     <joint name="chassis_battery_joint" type="fixed">
@@ -50,7 +44,6 @@
             <origin xyz="0 0 0.009" rpy="0 0 0" />
         </collision>
-        <!-- TODO simple approximation; needs correction -->
-        <xacro:box_inertia m="0.15" l="0.138" w="0.045" h="0.018"
-            xyz="-0.069 -0.0225 0" rpy="0 0 0" />
+        <xacro:box_inertia m="0.35" l="0.138" w="0.045" h="0.018"
+            xyz="0 0 0.009" rpy="0 0 0" />
     </link>
     <joint name="chassis_raspberry_joint" type="fixed">
@@ -74,7 +67,6 @@
             <origin xyz="0 0 0.0125" rpy="0 0 0" />
         </collision>
-        <!-- TODO simple approximation; needs correction -->
-        <xacro:box_inertia m="0.35" l="0.1" w="0.07" h="0.025"
-            xyz="-0.05 -0.035 0" rpy="0 0 0" />
+        <xacro:box_inertia m="0.15" l="0.1" w="0.07" h="0.025"
+            xyz="0 0 0.0125" rpy="0 0 0" />
     </link>
 </robot>

File: qronk_description/urdf/common_properties.xacro (robot description, xacro)
@@ -24,13 +24,4 @@
         </inertial>
     </xacro:macro>
-    <xacro:macro name="cylinder_inertia" params="m r l xyz rpy">
-        <inertial>
-            <origin xyz="${xyz}" rpy="${rpy}" />
-            <mass value="${m}" />
-            <inertia ixx="${m * (3 * r**2 + l**2) / 12.0}" ixy="0" ixz="0"
-                iyy="${m * (3 * r**2 + l**2) / 12.0}" iyz="0"
-                izz="${m * r**2 / 2.0}" />
-        </inertial>
-    </xacro:macro>
     <xacro:macro name="sphere_inertia" params="m r xyz rpy">
         <inertial>

File: qronk_description/urdf/leg_BL.xacro (robot description, xacro)
@@ -1,6 +1,6 @@
 <?xml version="1.0"?>
 <robot xmlns:xacro="http://www.ros.org/wiki/xacro">
-    <joint name="base_shoulder_BL_joint" type="revolute">
-        <parent link="base_link" />
+    <joint name="chassis_shoulder_BL_joint" type="revolute">
+        <parent link="chassis_link" />
         <child link="shoulder_BL_link" />
         <origin xyz="-0.0885 0.047417 0.000052" rpy="0 0 0" />
@@ -17,4 +17,12 @@
             <material name="grey" />
         </visual>
+        <collision>
+            <geometry>
+                <box size="0.05 0.04 0.068" />
+            </geometry>
+            <origin xyz="-0.03 -0 -0.005" rpy="0 0 0" />
+        </collision>
+        <xacro:box_inertia m="0.1" l="0.05" w="0.04" h="0.068"
+            xyz="-0.03 -0 -0.005" rpy="0 0 0" />
     </link>
     <joint name="shoulder_upper_leg_BL_joint" type="revolute">
@@ -34,4 +42,12 @@
             <material name="grey" />
         </visual>
+        <collision>
+            <geometry>
+                <box size="0.05 0.0532 0.137" />
+            </geometry>
+            <origin xyz="-0 0.0266 -0.0435" rpy="0 0 0" />
+        </collision>
+        <xacro:box_inertia m="0.1" l="0.05" w="0.0532" h="0.0137"
+            xyz="-0 0.0266 -0.0435" rpy="0 0 0" />
     </link>
     <joint name="upper_leg_lower_leg_BL_joint" type="revolute">
@@ -51,4 +67,12 @@
             <material name="grey" />
         </visual>
+        <collision>
+            <geometry>
+                <box size="0.028 0.0134 0.102" />
+            </geometry>
+            <origin xyz="-0 0.0067 -0.037" rpy="0 0 0" />
+        </collision>
+        <xacro:box_inertia m="0.1" l="0.028" w="0.0134" h="0.102"
+            xyz="-0 0.0067 -0.037" rpy="0 0 0" />
     </link>
     <joint name="lower_leg_foot_BL_joint" type="fixed">
@@ -65,4 +89,12 @@
             <material name="grey" />
         </visual>
+        <collision>
+            <geometry>
+                <sphere radius="0.0075" />
+            </geometry>
+            <origin xyz="0 0 0" rpy="0 0 0" />
+        </collision>
+        <xacro:sphere_inertia m="0.05" r="0.0075"
+            xyz="0 0 0" rpy="0 0 0" />
     </link>
 </robot>

File: qronk_description/urdf/leg_BR.xacro (robot description, xacro)
@@ -1,6 +1,6 @@
 <?xml version="1.0"?>
 <robot xmlns:xacro="http://www.ros.org/wiki/xacro">
-    <joint name="base_shoulder_BR_joint" type="revolute">
-        <parent link="base_link" />
+    <joint name="chassis_shoulder_BR_joint" type="revolute">
+        <parent link="chassis_link" />
         <child link="shoulder_BR_link" />
         <origin xyz="-0.0885 -0.047417 0.000052" rpy="0 0 0" />
@@ -17,4 +17,12 @@
             <material name="grey" />
         </visual>
+        <collision>
+            <geometry>
+                <box size="0.05 0.04 0.068" />
+            </geometry>
+            <origin xyz="-0.03 0 -0.005" rpy="0 0 0" />
+        </collision>
+        <xacro:box_inertia m="0.1" l="0.05" w="0.04" h="0.068"
+            xyz="-0.03 0 -0.005" rpy="0 0 0" />
     </link>
     <joint name="shoulder_upper_leg_BR_joint" type="revolute">
@@ -34,4 +42,12 @@
             <material name="grey" />
         </visual>
+        <collision>
+            <geometry>
+                <box size="0.05 0.0532 0.137" />
+            </geometry>
+            <origin xyz="-0 -0.0266 -0.0435" rpy="0 0 0" />
+        </collision>
+        <xacro:box_inertia m="0.1" l="0.05" w="0.0532" h="0.0137"
+            xyz="-0 -0.0266 -0.0435" rpy="0 0 0" />
     </link>
     <joint name="upper_leg_lower_leg_BR_joint" type="revolute">
@@ -51,4 +67,12 @@
             <material name="grey" />
         </visual>
+        <collision>
+            <geometry>
+                <box size="0.028 0.0134 0.102" />
+            </geometry>
+            <origin xyz="-0 -0.0067 -0.037" rpy="0 0 0" />
+        </collision>
+        <xacro:box_inertia m="0.1" l="0.028" w="0.0134" h="0.102"
+            xyz="-0 -0.0067 -0.037" rpy="0 0 0" />
     </link>
     <joint name="lower_leg_foot_BR_joint" type="fixed">
@@ -65,4 +89,12 @@
             <material name="grey" />
         </visual>
+        <collision>
+            <geometry>
+                <sphere radius="0.0075" />
+            </geometry>
+            <origin xyz="0 0 0" rpy="0 0 0" />
+        </collision>
+        <xacro:sphere_inertia m="0.05" r="0.0075"
+            xyz="0 0 0" rpy="0 0 0" />
     </link>
 </robot>

File: qronk_description/urdf/leg_FL.xacro (robot description, xacro)
@@ -1,6 +1,6 @@
 <?xml version="1.0"?>
 <robot xmlns:xacro="http://www.ros.org/wiki/xacro">
-    <joint name="base_shoulder_FL_joint" type="revolute">
-        <parent link="base_link" />
+    <joint name="chassis_shoulder_FL_joint" type="revolute">
+        <parent link="chassis_link" />
         <child link="shoulder_FL_link" />
         <origin xyz="0.0885 0.047417 0.000052" rpy="0 0 0" />
@@ -17,4 +17,12 @@
             <material name="grey" />
         </visual>
+        <collision>
+            <geometry>
+                <box size="0.05 0.04 0.068" />
+            </geometry>
+            <origin xyz="0.03 -0 -0.005" rpy="0 0 0" />
+        </collision>
+        <xacro:box_inertia m="0.1" l="0.05" w="0.04" h="0.068"
+            xyz="0.03 -0 -0.005" rpy="0 0 0" />
     </link>
     <joint name="shoulder_upper_leg_FL_joint" type="revolute">
@@ -34,4 +42,12 @@
             <material name="grey" />
         </visual>
+        <collision>
+            <geometry>
+                <box size="0.05 0.0532 0.137" />
+            </geometry>
+            <origin xyz="0 0.0266 -0.0435" rpy="0 0 0" />
+        </collision>
+        <xacro:box_inertia m="0.1" l="0.05" w="0.0532" h="0.0137"
+            xyz="0 0.0266 -0.0435" rpy="0 0 0" />
     </link>
     <joint name="upper_leg_lower_leg_FL_joint" type="revolute">
@@ -51,4 +67,12 @@
             <material name="grey" />
         </visual>
+        <collision>
+            <geometry>
+                <box size="0.028 0.0134 0.102" />
+            </geometry>
+            <origin xyz="0 0.0067 -0.037" rpy="0 0 0" />
+        </collision>
+        <xacro:box_inertia m="0.1" l="0.028" w="0.0134" h="0.102"
+            xyz="0 0.0067 -0.037" rpy="0 0 0" />
     </link>
     <joint name="lower_leg_foot_FL_joint" type="fixed">
@@ -65,4 +89,12 @@
             <material name="grey" />
         </visual>
+        <collision>
+            <geometry>
+                <sphere radius="0.0075" />
+            </geometry>
+            <origin xyz="0 0 0" rpy="0 0 0" />
+        </collision>
+        <xacro:sphere_inertia m="0.05" r="0.0075"
+            xyz="0 0 0" rpy="0 0 0" />
     </link>
 </robot>

File: qronk_description/urdf/leg_FR.xacro (robot description, xacro)
@@ -1,6 +1,6 @@
 <?xml version="1.0"?>
 <robot xmlns:xacro="http://www.ros.org/wiki/xacro">
-    <joint name="base_shoulder_FR_joint" type="revolute">
-        <parent link="base_link" />
+    <joint name="chassis_shoulder_FR_joint" type="revolute">
+        <parent link="chassis_link" />
         <child link="shoulder_FR_link" />
         <origin xyz="0.0885 -0.047417 0.000052" rpy="0 0 0" />
@@ -17,4 +17,12 @@
             <material name="grey" />
         </visual>
+        <collision>
+            <geometry>
+                <box size="0.05 0.04 0.068" />
+            </geometry>
+            <origin xyz="0.03 0 -0.005" rpy="0 0 0" />
+        </collision>
+        <xacro:box_inertia m="0.1" l="0.05" w="0.04" h="0.068"
+            xyz="0.03 0 -0.005" rpy="0 0 0" />
     </link>
     <joint name="shoulder_upper_leg_FR_joint" type="revolute">
@@ -34,4 +42,12 @@
             <material name="grey" />
         </visual>
+        <collision>
+            <geometry>
+                <box size="0.05 0.0532 0.137" />
+            </geometry>
+            <origin xyz="0 -0.0266 -0.0435" rpy="0 0 0" />
+        </collision>
+        <xacro:box_inertia m="0.1" l="0.05" w="0.0532" h="0.0137"
+            xyz="0 -0.0266 -0.0435" rpy="0 0 0" />
     </link>
     <joint name="upper_leg_lower_leg_FR_joint" type="revolute">
@@ -51,4 +67,12 @@
             <material name="grey" />
         </visual>
+        <collision>
+            <geometry>
+                <box size="0.028 0.0134 0.102" />
+            </geometry>
+            <origin xyz="0 -0.0067 -0.037" rpy="0 0 0" />
+        </collision>
+        <xacro:box_inertia m="0.1" l="0.028" w="0.0134" h="0.102"
+            xyz="0 -0.0067 -0.037" rpy="0 0 0" />
     </link>
     <joint name="lower_leg_foot_FR_joint" type="fixed">
@@ -65,4 +89,12 @@
             <material name="grey" />
         </visual>
+        <collision>
+            <geometry>
+                <sphere radius="0.0075" />
+            </geometry>
+            <origin xyz="0 0 0" rpy="0 0 0" />
+        </collision>
+        <xacro:sphere_inertia m="0.05" r="0.0075"
+            xyz="0 0 0" rpy="0 0 0" />
     </link>
 </robot>

File: qronk_description/urdf/qronk.urdf.xacro (robot description, xacro)
@@ -4,12 +4,8 @@
     <xacro:include filename="common_properties.xacro" />
     <xacro:include filename="chassis.xacro" />
-    <xacro:include filename="chassis_gazebo.xacro" />
     <xacro:include filename="leg_FR.xacro" />
-    <xacro:include filename="leg_FR_gazebo.xacro" />
     <xacro:include filename="leg_FL.xacro" />
-    <xacro:include filename="leg_FL_gazebo.xacro" />
     <xacro:include filename="leg_BR.xacro" />
-    <xacro:include filename="leg_BR_gazebo.xacro" />
     <xacro:include filename="leg_BL.xacro" />
-    <xacro:include filename="leg_BL_gazebo.xacro" />
+    <xacro:include filename="qronk_gazebo.xacro" />
 </robot>

Commit message: Updated xacro files, supports both Gazebo and RVIZ

File: qronk_description/urdf/chassis.xacro (robot description, xacro)
@@ -1,4 +1,5 @@
 <?xml version="1.0"?>
 <robot xmlns:xacro="http://www.ros.org/wiki/xacro">
+<!--Updated all model xacros to be compatible with rvis and gazebo-->
     <joint name="base_chassis_joint" type="fixed">
         <parent link="base_link" />
@@ -9,5 +10,5 @@
         <visual>
             <geometry>
-                <mesh filename="package://qronk_description/meshes/chassis.stl"
+                <mesh filename="file://$(find qronk_description)/meshes/chassis.stl"
                     scale="0.001 0.001 0.001" />
             </geometry>
@@ -32,5 +33,5 @@
         <visual>
             <geometry>
-                <mesh filename="package://qronk_description/meshes/battery.stl"
+                <mesh filename="file://$(find qronk_description)/meshes/battery.stl"
                     scale="0.001 0.001 0.001" />
             </geometry>
@@ -55,5 +56,5 @@
         <visual>
             <geometry>
-                <mesh filename="package://qronk_description/meshes/raspberry.stl"
+                <mesh filename="file://$(find qronk_description)/meshes/raspberry.stl"
                     scale="0.001 0.001 0.001" />
             </geometry>

File: qronk_description/urdf/leg_BL.xacro (robot description, xacro)
@@ -11,5 +11,5 @@
         <visual>
             <geometry>
-                <mesh filename="package://qronk_description/meshes/shoulder_BL.stl"
+                <mesh filename="file://$(find qronk_description)/meshes/shoulder_BL.stl"
                     scale="0.001 0.001 0.001" />
             </geometry>
@@ -36,5 +36,5 @@
         <visual>
             <geometry>
-                <mesh filename="package://qronk_description/meshes/upper_leg_BL.stl"
+                <mesh filename="file://$(find qronk_description)/meshes/upper_leg_BL.stl"
                     scale="0.001 0.001 0.001" />
             </geometry>
@@ -61,5 +61,5 @@
         <visual>
             <geometry>
-                <mesh filename="package://qronk_description/meshes/lower_leg_BL.stl"
+                <mesh filename="file://$(find qronk_description)/meshes/lower_leg_BL.stl"
                     scale="0.001 0.001 0.001" />
             </geometry>

File: qronk_description/urdf/leg_BR.xacro (robot description, xacro)
@@ -11,5 +11,5 @@
         <visual>
             <geometry>
-                <mesh filename="package://qronk_description/meshes/shoulder_BR.stl"
+                <mesh filename="file://$(find qronk_description)/meshes/shoulder_BR.stl"
                     scale="0.001 0.001 0.001" />
             </geometry>
@@ -36,5 +36,5 @@
         <visual>
             <geometry>
-                <mesh filename="package://qronk_description/meshes/upper_leg_BR.stl"
+                <mesh filename="file://$(find qronk_description)/meshes/upper_leg_BR.stl"
                     scale="0.001 0.001 0.001" />
             </geometry>
@@ -61,5 +61,5 @@
         <visual>
             <geometry>
-                <mesh filename="package://qronk_description/meshes/lower_leg_BR.stl"
+                <mesh filename="file://$(find qronk_description)/meshes/lower_leg_BR.stl"
                     scale="0.001 0.001 0.001" />
             </geometry>

File: qronk_description/urdf/leg_FL.xacro (robot description, xacro)
@@ -11,5 +11,5 @@
         <visual>
             <geometry>
-                <mesh filename="package://qronk_description/meshes/shoulder_FL.stl"
+                <mesh filename="file://$(find qronk_description)/meshes/shoulder_FL.stl"
                     scale="0.001 0.001 0.001" />
             </geometry>
@@ -36,5 +36,5 @@
         <visual>
             <geometry>
-                <mesh filename="package://qronk_description/meshes/upper_leg_FL.stl"
+                <mesh filename="file://$(find qronk_description)/meshes/upper_leg_FL.stl"
                     scale="0.001 0.001 0.001" />
             </geometry>
@@ -61,5 +61,5 @@
         <visual>
             <geometry>
-                <mesh filename="package://qronk_description/meshes/lower_leg_FL.stl"
+                <mesh filename="file://$(find qronk_description)/meshes/lower_leg_FL.stl"
                     scale="0.001 0.001 0.001" />
             </geometry>

File: qronk_description/urdf/leg_FR.xacro (robot description, xacro)
@@ -11,5 +11,5 @@
         <visual>
             <geometry>
-                <mesh filename="package://qronk_description/meshes/shoulder_FR.stl"
+                <mesh filename="file://$(find qronk_description)/meshes/shoulder_FR.stl"
                     scale="0.001 0.001 0.001" />
             </geometry>
@@ -36,5 +36,5 @@
         <visual>
             <geometry>
-                <mesh filename="package://qronk_description/meshes/upper_leg_FR.stl"
+                <mesh filename="file://$(find qronk_description)//meshes/upper_leg_FR.stl"
                     scale="0.001 0.001 0.001" />
             </geometry>
@@ -61,5 +61,5 @@
         <visual>
             <geometry>
-                <mesh filename="package://qronk_description/meshes/lower_leg_FR.stl"
+                <mesh filename="file://$(find qronk_description)//meshes/lower_leg_FR.stl"
                     scale="0.001 0.001 0.001" />
             </geometry>
