Commit message: Created a qronk_pybullet package

File: qronk_pybullet_OLD/qronk.urdf (robot description, URDF)
Before this commit: robot qronk, 20 links, 19 joints
Links:
- link battery_link: geometry collision box size=0.138 0.045 0.018; visual mesh filename=package://qronk_description/meshes/battery.stl scale=0.001 0.001 0.001
- link chassis_link: geometry collision box size=0.185 0.136835 0.084144; visual mesh filename=package://qronk_description/meshes/chassis.stl scale=0.001 0.001 0.001
- link lower_leg_BL_link: geometry collision box size=0.028 0.0134 0.102; visual mesh filename=package://qronk_description/meshes/lower_leg_BL.stl scale=0.001 0.001 0.001
- link lower_leg_BR_link: geometry collision box size=0.028 0.0134 0.102; visual mesh filename=package://qronk_description/meshes/lower_leg_BR.stl scale=0.001 0.001 0.001
- link lower_leg_FL_link: geometry collision box size=0.028 0.0134 0.102; visual mesh filename=package://qronk_description/meshes/lower_leg_FL.stl scale=0.001 0.001 0.001
- link lower_leg_FR_link: geometry collision box size=0.028 0.0134 0.102; visual mesh filename=package://qronk_description/meshes/lower_leg_FR.stl scale=0.001 0.001 0.001
- link raspberry_link: geometry collision box size=0.1 0.07 0.025; visual mesh filename=package://qronk_description/meshes/raspberry.stl scale=0.001 0.001 0.001
- link shoulder_BL_link: geometry collision box size=0.05 0.04 0.068; visual mesh filename=package://qronk_description/meshes/shoulder_BL.stl scale=0.001 0.001 0.001
- link shoulder_BR_link: geometry collision box size=0.05 0.04 0.068; visual mesh filename=package://qronk_description/meshes/shoulder_BR.stl scale=0.001 0.001 0.001
- link shoulder_FL_link: geometry collision box size=0.05 0.04 0.068; visual mesh filename=package://qronk_description/meshes/shoulder_FL.stl scale=0.001 0.001 0.001
- link shoulder_FR_link: geometry collision box size=0.05 0.04 0.068; visual mesh filename=package://qronk_description/meshes/shoulder_FR.stl scale=0.001 0.001 0.001
- link upper_leg_BL_link: geometry collision box size=0.05 0.0532 0.137; visual mesh filename=package://qronk_description/meshes/upper_leg_BL.stl scale=0.001 0.001 0.001
- link upper_leg_BR_link: geometry collision box size=0.05 0.0532 0.137; visual mesh filename=package://qronk_description/meshes/upper_leg_BR.stl scale=0.001 0.001 0.001
- link upper_leg_FL_link: geometry collision box size=0.05 0.0532 0.137; visual mesh filename=package://qronk_description/meshes/upper_leg_FL.stl scale=0.001 0.001 0.001
- link upper_leg_FR_link: geometry collision box size=0.05 0.0532 0.137; visual mesh filename=package://qronk_description/meshes/upper_leg_FR.stl scale=0.001 0.001 0.001
